Commit message: Add files via upload

File: urdf/smr100e2_description.urdf (robot description, URDF)
Before this commit: robot smr100e2_description, 22 links, 21 joints
Links:
- link base_link: mass 26.046 -> 31.222
- link caster_front_left_wheel_link: mass 0.10623 -> 0.10622773912148
- link caster_front_right_arm_link: mass 0.11891 -> 0.118905856919371
- link caster_front_right_wheel_link: mass 0.10623 -> 0.106227739121479
- link caster_rear_left_arm_link: mass 0.11891 -> 0.11890585691937
- link caster_rear_left_wheel_link: mass 0.10623 -> 0.106227739121479
- link caster_rear_right_arm_link: mass 0.11891 -> 0.118905856919369
- link caster_rear_right_wheel_link: mass 0.10623 -> 0.10622773912148
- link imu_link: mass 0.00091136 -> 0.000911356888660493
- link lidar_front_right_link: mass 0.096744 -> 0.096744416647924
- link lidar_rear_left_link: mass 0.096744 -> 0.0967444166479226
- link ultrasonic_front_left_link: mass 0.0086236 -> 0.00862358242165747
- link ultrasonic_front_left_side_link: mass 0.0086236 -> 0.00862358242165751
- link ultrasonic_front_right_link: mass 0.0086236 -> 0.00862358242165747
- link ultrasonic_front_right_side_link: mass 0.0086236 -> 0.00862358242165751
- link ultrasonic_rear_left_link: mass 0.0086236 -> 0.00862358242165748
- link ultrasonic_rear_left_side_link: mass 0.0086236 -> 0.00862358242165751
- link ultrasonic_rear_right_link: mass 0.0086236 -> 0.00862358242165749
- link ultrasonic_rear_right_side_link: mass 0.0086236 -> 0.0086235824216575
- link wheel_right_link: mass 4.9554 -> 4.95544635924953
Joints:
- joint caster_front_left_arm_joint: origin xyz=0.3725 0.155 0.10942 rpy=0 0 0 -> xyz=0.3725 0.155 0.11 rpy=0 0 0
- joint caster_front_right_arm_joint: origin xyz=0.3725 -0.155 0.10942 rpy=0 0 0 -> xyz=0.3725 -0.155 0.11 rpy=0 0 0
- joint caster_rear_left_arm_joint: origin xyz=-0.3725 0.155 0.10942 rpy=0 0 0 -> xyz=-0.3725 0.155 0.11 rpy=0 0 0
- joint caster_rear_right_arm_joint: origin xyz=-0.3725 -0.155 0.10942 rpy=0 0 0 -> xyz=-0.3725 -0.155 0.11 rpy=0 0 0
- joint imu_joint: origin xyz=0.061 0.0025 0.25852 rpy=0 0 -1.5708 -> xyz=0.061 0.0025 0.2591 rpy=0 0 -1.5708
- joint lidar_front_right_joint: origin xyz=0.4425 0 0.15277 rpy=0 0 0 -> xyz=0.4425 0 0.15335 rpy=0 0 0
- joint lidar_rear_left_joint: origin xyz=-0.4425 0 0.15277 rpy=0 0 3.1416 -> xyz=-0.4425 0 0.15335 rpy=0 0 3.1416
- joint ultrasonic_front_left_link: origin xyz=0.4967 0.1507 0.31042 rpy=0 0 0 -> xyz=0.4967 0.1507 0.311 rpy=0 0 0
- joint ultrasonic_front_left_side_joint: origin xyz=0.2528 0.2537 0.31092 rpy=0 0 1.5708 -> xyz=0.2528 0.2537 0.3115 rpy=0 0 1.5708
- joint ultrasonic_front_right_right: origin xyz=0.4967 -0.1493 0.31042 rpy=0 0 0 -> xyz=0.4967 -0.1493 0.311 rpy=0 0 0
- joint ultrasonic_front_right_side_joint: origin xyz=0.2522 -0.2517 0.31092 rpy=0 0 -1.5708 -> xyz=0.2522 -0.2517 0.3115 rpy=0 0 -1.5708
- joint ultrasonic_rear_left_joint: origin xyz=-0.4902 0.1513 0.32592 rpy=0 0 3.1416 -> xyz=-0.4902 0.1513 0.3265 rpy=0 0 3.1416
- joint ultrasonic_rear_left_side_link: origin xyz=-0.2872 0.2537 0.31092 rpy=0 0 1.5708 -> xyz=-0.2872 0.2537 0.3115 rpy=0 0 1.5708
- joint ultrasonic_rear_right_joint: origin xyz=-0.4902 -0.1487 0.32592 rpy=0 0 3.1416 -> xyz=-0.4902 -0.1487 0.3265 rpy=0 0 3.1416
- joint ultrasonic_rear_right_side_joint: origin xyz=-0.2878 -0.2517 0.31092 rpy=0 0 -1.5708 -> xyz=-0.2878 -0.2517 0.3115 rpy=0 0 -1.5708
- joint wheel_left_joint: axis 0 1 0 -> 0 -1 0; limit (none) -> effort=0 velocity=21
- joint wheel_right_joint: limit (none) -> effort=0 velocity=21
